Commit message: feat: calibrate Pivot-G2 control and robot hardware

File: src/vacuum_robot_gazebo/urdf/vacuum_robot.urdf (robot description, URDF)
Before this commit: robot vacuum_robot, 6 links, 5 joints
Links:
- added link left_motor; visual cylinder length=0.068 radius=0.0125
- added link right_motor; visual cylinder length=0.068 radius=0.0125
Joints:
- added joint base_to_left_motor: type fixed, parent base_link, child left_motor, origin xyz=0 0.0934 0 rpy=0 0 0
- added joint base_to_right_motor: type fixed, parent base_link, child right_motor, origin xyz=0 -0.0934 0 rpy=0 0 0
- joint left_wheel_joint: limit effort=20 velocity=10 -> effort=0.3530394 velocity=13.6135681656
- joint right_wheel_joint: limit effort=20 velocity=10 -> effort=0.3530394 velocity=13.6135681656
